File: Nauka_120-degrees_control.kicad_pcb (KiCad board)
At the start: 2 copper layers, 33.2 x 36.5 mm, 21 parts, among them U1 4040, U2 4017, Y1 4.9152M

Commit message: VER1.0: добавил драйвера
Parts:
- removed D2: ~, Package_SO:SOIC-14_3.9x8.7mm_P1.27mm
- added C10: 10u, Capacitor_SMD:C_1206_3216Metric_Pad1.33x1.80mm_HandSolder, F.Cu at (152.1, 160.7)
- added C11: 10u, Capacitor_SMD:C_1206_3216Metric_Pad1.33x1.80mm_HandSolder, F.Cu at (152.1, 164.0)
- added C13: 2.2u, Capacitor_SMD:C_0805_2012Metric_Pad1.18x1.45mm_HandSolder, F.Cu at (196.5, 116.6)
- added C14: 100p, Capacitor_SMD:C_0805_2012Metric_Pad1.18x1.45mm_HandSolder, F.Cu at (196.5, 119.6)
- added C15: 4.7u, Capacitor_SMD:C_1206_3216Metric_Pad1.33x1.80mm_HandSolder, F.Cu at (238.0, 136.5)
- added C16: 4.7u, Capacitor_SMD:C_1206_3216Metric_Pad1.33x1.80mm_HandSolder, F.Cu at (238.0, 139.8)
- added C17: 10n, Capacitor_SMD:C_0805_2012Metric_Pad1.18x1.45mm_HandSolder, F.Cu at (196.5, 122.7)
- added C18: 10u, Capacitor_SMD:C_1206_3216Metric_Pad1.33x1.80mm_HandSolder, F.Cu at (158.1, 154.0)
- added C19: 10u, Capacitor_SMD:C_1206_3216Metric_Pad1.33x1.80mm_HandSolder, F.Cu at (158.1, 157.3)
- added C20: 4.7u, Capacitor_SMD:C_1206_3216Metric_Pad1.33x1.80mm_HandSolder, F.Cu at (158.1, 160.7)
- added C21: 4.7u, Capacitor_SMD:C_1206_3216Metric_Pad1.33x1.80mm_HandSolder, F.Cu at (158.1, 164.0)
- added C22: 10u, Capacitor_SMD:C_1206_3216Metric_Pad1.33x1.80mm_HandSolder, F.Cu at (164.1, 154.0)
- added C23: 10u, Capacitor_SMD:C_1206_3216Metric_Pad1.33x1.80mm_HandSolder, F.Cu at (164.1, 157.3)
- added C24: 2.2u, Capacitor_SMD:C_0805_2012Metric_Pad1.18x1.45mm_HandSolder, F.Cu at (196.5, 125.7)
- added C25: 100p, Capacitor_SMD:C_0805_2012Metric_Pad1.18x1.45mm_HandSolder, F.Cu at (196.5, 128.7)
- added C26: 10n, Capacitor_SMD:C_0805_2012Metric_Pad1.18x1.45mm_HandSolder, F.Cu at (201.3, 113.6)
- added C27: 56p, Capacitor_SMD:C_0805_2012Metric_Pad1.18x1.45mm_HandSolder, F.Cu at (201.3, 116.6)
- added C28: 56p, Capacitor_SMD:C_0805_2012Metric_Pad1.18x1.45mm_HandSolder, F.Cu at (201.3, 119.6)
- added C29: 10u, Capacitor_SMD:C_1206_3216Metric_Pad1.33x1.80mm_HandSolder, F.Cu at (164.1, 160.7)
- added C30: 10u, Capacitor_SMD:C_1206_3216Metric_Pad1.33x1.80mm_HandSolder, F.Cu at (164.1, 164.0)
- added C31: 56p, Capacitor_SMD:C_0805_2012Metric_Pad1.18x1.45mm_HandSolder, F.Cu at (201.3, 122.7)
- added C32: 56p, Capacitor_SMD:C_0805_2012Metric_Pad1.18x1.45mm_HandSolder, F.Cu at (201.3, 125.7)
- added C33: 10u, Capacitor_SMD:C_1206_3216Metric_Pad1.33x1.80mm_HandSolder, F.Cu at (238.0, 143.2)
- added C34: 10u, Capacitor_SMD:C_1206_3216Metric_Pad1.33x1.80mm_HandSolder, F.Cu at (238.0, 146.5)
- added C35: 2.2u, Capacitor_SMD:C_0805_2012Metric_Pad1.18x1.45mm_HandSolder, F.Cu at (261.4, 136.3)
- added C36: 100p, Capacitor_SMD:C_0805_2012Metric_Pad1.18x1.45mm_HandSolder, F.Cu at (261.4, 139.3)
- added C37: 56p, Capacitor_SMD:C_0805_2012Metric_Pad1.18x1.45mm_HandSolder, F.Cu at (261.4, 142.3)
- added C38: 10n, Capacitor_SMD:C_0805_2012Metric_Pad1.18x1.45mm_HandSolder, F.Cu at (261.4, 145.3)
- added C39: 10u, Capacitor_SMD:C_1206_3216Metric_Pad1.33x1.80mm_HandSolder, F.Cu at (238.0, 149.9)
- added C4: 100n, Capacitor_SMD:C_0805_2012Metric_Pad1.18x1.45mm_HandSolder, F.Cu at (196.5, 113.6)
- added C40: 10u, Capacitor_SMD:C_1206_3216Metric_Pad1.33x1.80mm_HandSolder, F.Cu at (238.0, 153.2)
- added C41: 56p, Capacitor_SMD:C_0805_2012Metric_Pad1.18x1.45mm_HandSolder, F.Cu at (261.4, 148.3)
- added C42: 4.7u, Capacitor_SMD:C_1206_3216Metric_Pad1.33x1.80mm_HandSolder, F.Cu at (244.0, 136.5)
- added C43: 4.7u, Capacitor_SMD:C_1206_3216Metric_Pad1.33x1.80mm_HandSolder, F.Cu at (244.0, 139.8)
- added C44: 10u, Capacitor_SMD:C_1206_3216Metric_Pad1.33x1.80mm_HandSolder, F.Cu at (244.0, 143.2)
- added C45: 10u, Capacitor_SMD:C_1206_3216Metric_Pad1.33x1.80mm_HandSolder, F.Cu at (244.0, 146.5)
- added C46: 2.2u, Capacitor_SMD:C_0805_2012Metric_Pad1.18x1.45mm_HandSolder, F.Cu at (266.2, 136.3)
- added C47: 100p, Capacitor_SMD:C_0805_2012Metric_Pad1.18x1.45mm_HandSolder, F.Cu at (266.2, 139.3)
- added C48: 10n, Capacitor_SMD:C_0805_2012Metric_Pad1.18x1.45mm_HandSolder, F.Cu at (266.2, 142.3)
- added C49: 56p, Capacitor_SMD:C_0805_2012Metric_Pad1.18x1.45mm_HandSolder, F.Cu at (266.2, 145.3)
- added C50: 10u, Capacitor_SMD:C_1206_3216Metric_Pad1.33x1.80mm_HandSolder, F.Cu at (244.0, 149.9)
- added C51: 10u, Capacitor_SMD:C_1206_3216Metric_Pad1.33x1.80mm_HandSolder, F.Cu at (244.0, 153.2)
- added C52: 56p, Capacitor_SMD:C_0805_2012Metric_Pad1.18x1.45mm_HandSolder, F.Cu at (266.2, 148.3)
- added C53: 4.7u, Capacitor_SMD:C_1206_3216Metric_Pad1.33x1.80mm_HandSolder, F.Cu at (250.0, 136.5)
- added C54: 4.7u, Capacitor_SMD:C_1206_3216Metric_Pad1.33x1.80mm_HandSolder, F.Cu at (250.0, 139.8)
- added C55: 10u, Capacitor_SMD:C_1206_3216Metric_Pad1.33x1.80mm_HandSolder, F.Cu at (250.0, 143.2)
- added C56: 10u, Capacitor_SMD:C_1206_3216Metric_Pad1.33x1.80mm_HandSolder, F.Cu at (250.0, 146.5)
- added C57: 2.2u, Capacitor_SMD:C_0805_2012Metric_Pad1.18x1.45mm_HandSolder, F.Cu at (271.1, 136.3)
- added C58: 100p, Capacitor_SMD:C_0805_2012Metric_Pad1.18x1.45mm_HandSolder, F.Cu at (271.1, 139.3)
- added C59: 56p, Capacitor_SMD:C_0805_2012Metric_Pad1.18x1.45mm_HandSolder, F.Cu at (271.1, 142.3)
- added C6: 4.7u, Capacitor_SMD:C_1206_3216Metric_Pad1.33x1.80mm_HandSolder, F.Cu at (152.1, 154.0)
- added C60: 10n, Capacitor_SMD:C_0805_2012Metric_Pad1.18x1.45mm_HandSolder, F.Cu at (271.1, 145.3)
- added C61: 10u, Capacitor_SMD:C_1206_3216Metric_Pad1.33x1.80mm_HandSolder, F.Cu at (250.0, 149.9)
- added C62: 10u, Capacitor_SMD:C_1206_3216Metric_Pad1.33x1.80mm_HandSolder, F.Cu at (250.0, 153.2)
- added C63: 56p, Capacitor_SMD:C_0805_2012Metric_Pad1.18x1.45mm_HandSolder, F.Cu at (271.1, 148.3)
- added C64: 4.7u, Capacitor_SMD:C_1206_3216Metric_Pad1.33x1.80mm_HandSolder, F.Cu at (256.0, 136.5)
- added C65: 4.7u, Capacitor_SMD:C_1206_3216Metric_Pad1.33x1.80mm_HandSolder, F.Cu at (256.0, 139.8)
- added C66: 10u, Capacitor_SMD:C_1206_3216Metric_Pad1.33x1.80mm_HandSolder, F.Cu at (256.0, 143.2)
- added C67: 10u, Capacitor_SMD:C_1206_3216Metric_Pad1.33x1.80mm_HandSolder, F.Cu at (256.0, 146.5)
- added C68: 2.2u, Capacitor_SMD:C_0805_2012Metric_Pad1.18x1.45mm_HandSolder, F.Cu at (275.9, 136.3)
- added C69: 100p, Capacitor_SMD:C_0805_2012Metric_Pad1.18x1.45mm_HandSolder, F.Cu at (275.9, 139.3)
- added C7: 4.7u, Capacitor_SMD:C_1206_3216Metric_Pad1.33x1.80mm_HandSolder, F.Cu at (152.1, 157.3)
- added C70: 10n, Capacitor_SMD:C_0805_2012Metric_Pad1.18x1.45mm_HandSolder, F.Cu at (275.9, 142.3)
- added C71: 56p, Capacitor_SMD:C_0805_2012Metric_Pad1.18x1.45mm_HandSolder, F.Cu at (275.9, 145.3)
- added C72: 10u, Capacitor_SMD:C_1206_3216Metric_Pad1.33x1.80mm_HandSolder, F.Cu at (256.0, 149.9)
- added C73: 10u, Capacitor_SMD:C_1206_3216Metric_Pad1.33x1.80mm_HandSolder, F.Cu at (256.0, 153.2)
- added C74: 56p, Capacitor_SMD:C_0805_2012Metric_Pad1.18x1.45mm_HandSolder, F.Cu at (275.9, 148.3)
- added D10: NSI6651, Package_SO:SOIC-16W_7.5x10.3mm_P1.27mm, F.Cu at (213.7, 140.8)
- added D12: NSI6651, Package_SO:SOIC-16W_7.5x10.3mm_P1.27mm, F.Cu at (180.9, 159.9)
- added D13: D_Small, Diode_SMD:D_SMA_Handsoldering, F.Cu at (189.1, 123.5)
- added D14: D_Small, Diode_SMD:D_SMA_Handsoldering, F.Cu at (189.1, 128.0)
- added D15: ~, Diode_SMD:D_SOD-123, F.Cu at (190.3, 161.7)
- added D16: ~, LED_SMD:LED_0805_2012Metric_Pad1.15x1.40mm_HandSolder, F.Cu at (169.5, 153.8)
- added D17: ~, LED_SMD:LED_0805_2012Metric_Pad1.15x1.40mm_HandSolder, F.Cu at (169.5, 156.9)
- added D18: ~, LED_SMD:LED_0805_2012Metric_Pad1.15x1.40mm_HandSolder, F.Cu at (169.5, 159.9)
- added D19: ~, LED_SMD:LED_0805_2012Metric_Pad1.15x1.40mm_HandSolder, F.Cu at (169.5, 162.9)
- added D20: D_Small, Diode_SMD:D_SMA_Handsoldering, F.Cu at (225.2, 137.1)
- added D21: D_Small, Diode_SMD:D_SMA_Handsoldering, F.Cu at (225.2, 141.6)
- added D22: ~, LED_SMD:LED_0805_2012Metric_Pad1.15x1.40mm_HandSolder, F.Cu at (232.6, 136.3)
- added D23: ~, Diode_SMD:D_SOD-123, F.Cu at (274.9, 156.6)
- added D24: ~, LED_SMD:LED_0805_2012Metric_Pad1.15x1.40mm_HandSolder, F.Cu at (232.6, 139.3)
- added D26: NSI6651, Package_SO:SOIC-16W_7.5x10.3mm_P1.27mm, F.Cu at (213.7, 152.8)
- added D27: D_Small, Diode_SMD:D_SMA_Handsoldering, F.Cu at (225.2, 146.2)
- added D28: D_Small, Diode_SMD:D_SMA_Handsoldering, F.Cu at (225.2, 150.7)
- added D29: ~, LED_SMD:LED_0805_2012Metric_Pad1.15x1.40mm_HandSolder, F.Cu at (232.6, 142.4)
- added D3: ~, Package_SO:SO-14_3.9x8.65mm_P1.27mm, F.Cu at (161.8, 147.2)
- added D30: ~, Diode_SMD:D_SOD-123, F.Cu at (274.9, 159.9)
- added D31: ~, LED_SMD:LED_0805_2012Metric_Pad1.15x1.40mm_HandSolder, F.Cu at (232.6, 145.4)
- added D33: NSI6651, Package_SO:SOIC-16W_7.5x10.3mm_P1.27mm, F.Cu at (213.7, 164.7)
- added D34: D_Small, Diode_SMD:D_SMA_Handsoldering, F.Cu at (225.2, 155.3)
- added D35: D_Small, Diode_SMD:D_SMA_Handsoldering, F.Cu at (225.2, 159.8)
- added D36: ~, LED_SMD:LED_0805_2012Metric_Pad1.15x1.40mm_HandSolder, F.Cu at (232.6, 148.5)
- added D37: ~, Diode_SMD:D_SOD-123, F.Cu at (274.9, 163.3)
- added D38: ~, LED_SMD:LED_0805_2012Metric_Pad1.15x1.40mm_HandSolder, F.Cu at (232.6, 151.5)
- added D4: NSI6651, Package_SO:SOIC-16W_7.5x10.3mm_P1.27mm, F.Cu at (180.9, 148.0)
- added D40: NSI6651, Package_SO:SOIC-16W_7.5x10.3mm_P1.27mm, F.Cu at (213.7, 176.7)
- added D41: D_Small, Diode_SMD:D_SMA_Handsoldering, F.Cu at (225.2, 164.4)
- added D42: D_Small, Diode_SMD:D_SMA_Handsoldering, F.Cu at (225.2, 168.9)
- added D43: ~, LED_SMD:LED_0805_2012Metric_Pad1.15x1.40mm_HandSolder, F.Cu at (232.6, 154.5)
- added D44: ~, Diode_SMD:D_SOD-123, F.Cu at (274.9, 166.6)
- added D45: ~, LED_SMD:LED_0805_2012Metric_Pad1.15x1.40mm_HandSolder, F.Cu at (232.6, 157.6)
- added D5: D_Small, Diode_SMD:D_SMA_Handsoldering, F.Cu at (189.1, 114.4)
- added D6: D_Small, Diode_SMD:D_SMA_Handsoldering, F.Cu at (189.1, 118.9)
- added D7: ~, Package_SO:SOIC-14_3.9x8.7mm_P1.27mm, F.Cu at (170.2, 147.2)
- added D8: ~, Diode_SMD:D_SOD-123, F.Cu at (190.3, 158.4)
- added L1: 12u, Inductor_SMD:L_1210_3225Metric_Pad1.42x2.65mm_HandSolder, F.Cu at (187.0, 132.4)
- added L10: 47u, Inductor_SMD:L_1812_4532Metric_Pad1.30x3.40mm_HandSolder, F.Cu at (262.4, 167.3)
- added L11: 12u, Inductor_SMD:L_1210_3225Metric_Pad1.42x2.65mm_HandSolder, F.Cu at (269.0, 169.6)
- added L12: 47u, Inductor_SMD:L_1812_4532Metric_Pad1.30x3.40mm_HandSolder, F.Cu at (262.4, 172.2)
- added L2: 47u, Inductor_SMD:L_1812_4532Metric_Pad1.30x3.40mm_HandSolder, F.Cu at (197.7, 132.7)
- added L3: 12u, Inductor_SMD:L_1210_3225Metric_Pad1.42x2.65mm_HandSolder, F.Cu at (187.0, 136.6)
- added L4: 47u, Inductor_SMD:L_1812_4532Metric_Pad1.30x3.40mm_HandSolder, F.Cu at (197.7, 137.6)
- added L5: 12u, Inductor_SMD:L_1210_3225Metric_Pad1.42x2.65mm_HandSolder, F.Cu at (269.0, 157.0)
- added L6: 47u, Inductor_SMD:L_1812_4532Metric_Pad1.30x3.40mm_HandSolder, F.Cu at (262.4, 157.4)
- added L7: 12u, Inductor_SMD:L_1210_3225Metric_Pad1.42x2.65mm_HandSolder, F.Cu at (269.0, 161.2)
- added L8: 47u, Inductor_SMD:L_1812_4532Metric_Pad1.30x3.40mm_HandSolder, F.Cu at (262.4, 162.3)
- added L9: 12u, Inductor_SMD:L_1210_3225Metric_Pad1.42x2.65mm_HandSolder, F.Cu at (269.0, 165.4)
- added Q1: C2M0280120D, Package_TO_SOT_THT:TO-247-3_Horizontal_TabUp, F.Cu at (152.4, 115.1)
- added Q2: C2M0280120D, Package_TO_SOT_THT:TO-247-3_Horizontal_TabUp, F.Cu at (169.8, 115.1)
- added Q3: C2M0280120D, Package_TO_SOT_THT:TO-247-3_Horizontal_TabUp, F.Cu at (210.5, 108.0)
- added Q4: C2M0280120D, Package_TO_SOT_THT:TO-247-3_Horizontal_TabUp, F.Cu at (227.9, 108.0)
- added Q5: C2M0280120D, Package_TO_SOT_THT:TO-247-3_Horizontal_TabUp, F.Cu at (245.4, 108.0)
- added Q6: C2M0280120D, Package_TO_SOT_THT:TO-247-3_Horizontal_TabUp, F.Cu at (262.8, 108.0)
- added R10: 510, Resistor_SMD:R_0805_2012Metric_Pad1.20x1.40mm_HandSolder, F.Cu at (189.7, 143.4)
- added R11: 1k, Resistor_SMD:R_0805_2012Metric_Pad1.20x1.40mm_HandSolder, F.Cu at (189.7, 146.4)
- added R12: Rdesat, Resistor_SMD:R_0805_2012Metric_Pad1.20x1.40mm_HandSolder, F.Cu at (189.7, 149.3)
- added R13: 3, Resistor_SMD:R_0805_2012Metric_Pad1.20x1.40mm_HandSolder, F.Cu at (189.7, 152.3)
- added R14: 3, Resistor_SMD:R_0805_2012Metric_Pad1.20x1.40mm_HandSolder, F.Cu at (189.7, 155.2)
- added R15: 510, Resistor_SMD:R_0805_2012Metric_Pad1.20x1.40mm_HandSolder, F.Cu at (237.4, 156.4)
- added R16: 1k, Resistor_SMD:R_0805_2012Metric_Pad1.20x1.40mm_HandSolder, F.Cu at (237.4, 159.3)
- added R17: Rdesat, Resistor_SMD:R_0805_2012Metric_Pad1.20x1.40mm_HandSolder, F.Cu at (237.4, 162.3)
- added R18: 1k, Resistor_SMD:R_0805_2012Metric_Pad1.20x1.40mm_HandSolder, F.Cu at (237.4, 165.2)
- added R19: 10k, Resistor_SMD:R_0805_2012Metric_Pad1.20x1.40mm_HandSolder, F.Cu at (194.5, 143.4)
- added R20: 510, Resistor_SMD:R_0805_2012Metric_Pad1.20x1.40mm_HandSolder, F.Cu at (194.5, 146.4)
- added R21: 1k, Resistor_SMD:R_0805_2012Metric_Pad1.20x1.40mm_HandSolder, F.Cu at (194.5, 149.3)
- added R22: Rdesat, Resistor_SMD:R_0805_2012Metric_Pad1.20x1.40mm_HandSolder, F.Cu at (194.5, 152.3)
- added R23: 3, Resistor_SMD:R_0805_2012Metric_Pad1.20x1.40mm_HandSolder, F.Cu at (194.5, 155.2)
- added R24: 3, Resistor_SMD:R_0805_2012Metric_Pad1.20x1.40mm_HandSolder, F.Cu at (199.2, 143.4)
- added R25: 1k, Resistor_SMD:R_0805_2012Metric_Pad1.20x1.40mm_HandSolder, F.Cu at (199.2, 146.4)
- added R26: 10k, Resistor_SMD:R_0805_2012Metric_Pad1.20x1.40mm_HandSolder, F.Cu at (199.2, 149.3)
- added R27: 1k, Resistor_SMD:R_0805_2012Metric_Pad1.20x1.40mm_HandSolder, F.Cu at (199.2, 152.3)
- added R28: 560, Resistor_SMD:R_0805_2012Metric_Pad1.20x1.40mm_HandSolder, F.Cu at (199.2, 155.2)
- added R29: 10k, Resistor_SMD:R_0805_2012Metric_Pad1.20x1.40mm_HandSolder, F.Cu at (204.0, 143.4)
- added R30: 1k, Resistor_SMD:R_0805_2012Metric_Pad1.20x1.40mm_HandSolder, F.Cu at (204.0, 146.4)
- added R31: 10k, Resistor_SMD:R_0805_2012Metric_Pad1.20x1.40mm_HandSolder, F.Cu at (204.0, 149.3)
- added R32: 560, Resistor_SMD:R_0805_2012Metric_Pad1.20x1.40mm_HandSolder, F.Cu at (204.0, 152.3)
- added R33: 1k, Resistor_SMD:R_0805_2012Metric_Pad1.20x1.40mm_HandSolder, F.Cu at (204.0, 155.2)
- added R34: 3, Resistor_SMD:R_0805_2012Metric_Pad1.20x1.40mm_HandSolder, F.Cu at (237.4, 168.2)
- added R35: 3, Resistor_SMD:R_0805_2012Metric_Pad1.20x1.40mm_HandSolder, F.Cu at (237.4, 171.1)
- added R36: 10k, Resistor_SMD:R_0805_2012Metric_Pad1.20x1.40mm_HandSolder, F.Cu at (237.4, 174.1)
- added R37: 10k, Resistor_SMD:R_0805_2012Metric_Pad1.20x1.40mm_HandSolder, F.Cu at (237.4, 177.0)
- added R38: 560, Resistor_SMD:R_0805_2012Metric_Pad1.20x1.40mm_HandSolder, F.Cu at (242.1, 156.4)
- added R39: 1k, Resistor_SMD:R_0805_2012Metric_Pad1.20x1.40mm_HandSolder, F.Cu at (242.1, 159.3)
- added R40: 510, Resistor_SMD:R_0805_2012Metric_Pad1.20x1.40mm_HandSolder, F.Cu at (242.1, 162.3)
- added R41: 1k, Resistor_SMD:R_0805_2012Metric_Pad1.20x1.40mm_HandSolder, F.Cu at (242.1, 165.2)
- added R42: Rdesat, Resistor_SMD:R_0805_2012Metric_Pad1.20x1.40mm_HandSolder, F.Cu at (242.1, 168.2)
- added R43: 1k, Resistor_SMD:R_0805_2012Metric_Pad1.20x1.40mm_HandSolder, F.Cu at (242.1, 171.1)
- added R44: 3, Resistor_SMD:R_0805_2012Metric_Pad1.20x1.40mm_HandSolder, F.Cu at (242.1, 174.1)
- added R45: 3, Resistor_SMD:R_0805_2012Metric_Pad1.20x1.40mm_HandSolder, F.Cu at (242.1, 177.0)
- added R46: 10k, Resistor_SMD:R_0805_2012Metric_Pad1.20x1.40mm_HandSolder, F.Cu at (246.9, 156.4)
- added R47: 10k, Resistor_SMD:R_0805_2012Metric_Pad1.20x1.40mm_HandSolder, F.Cu at (246.9, 159.3)
- added R48: 560, Resistor_SMD:R_0805_2012Metric_Pad1.20x1.40mm_HandSolder, F.Cu at (246.9, 162.3)
- added R49: 1k, Resistor_SMD:R_0805_2012Metric_Pad1.20x1.40mm_HandSolder, F.Cu at (246.9, 165.2)
- added R50: 510, Resistor_SMD:R_0805_2012Metric_Pad1.20x1.40mm_HandSolder, F.Cu at (246.9, 168.2)
- added R51: 1k, Resistor_SMD:R_0805_2012Metric_Pad1.20x1.40mm_HandSolder, F.Cu at (246.9, 171.1)
- added R52: Rdesat, Resistor_SMD:R_0805_2012Metric_Pad1.20x1.40mm_HandSolder, F.Cu at (246.9, 174.1)
- added R53: 1k, Resistor_SMD:R_0805_2012Metric_Pad1.20x1.40mm_HandSolder, F.Cu at (246.9, 177.0)
- added R54: 3, Resistor_SMD:R_0805_2012Metric_Pad1.20x1.40mm_HandSolder, F.Cu at (251.6, 156.4)
- added R55: 3, Resistor_SMD:R_0805_2012Metric_Pad1.20x1.40mm_HandSolder, F.Cu at (251.6, 159.3)
- added R56: 10k, Resistor_SMD:R_0805_2012Metric_Pad1.20x1.40mm_HandSolder, F.Cu at (251.6, 162.3)
- added R57: 10k, Resistor_SMD:R_0805_2012Metric_Pad1.20x1.40mm_HandSolder, F.Cu at (251.6, 165.2)
- added R58: 560, Resistor_SMD:R_0805_2012Metric_Pad1.20x1.40mm_HandSolder, F.Cu at (251.6, 168.2)
- added R59: 1k, Resistor_SMD:R_0805_2012Metric_Pad1.20x1.40mm_HandSolder, F.Cu at (251.6, 171.1)
- added R60: 510, Resistor_SMD:R_0805_2012Metric_Pad1.20x1.40mm_HandSolder, F.Cu at (251.6, 174.1)
- added R61: 1k, Resistor_SMD:R_0805_2012Metric_Pad1.20x1.40mm_HandSolder, F.Cu at (251.6, 177.0)
- added R62: Rdesat, Resistor_SMD:R_0805_2012Metric_Pad1.20x1.40mm_HandSolder, F.Cu at (256.4, 156.4)
- added R63: 1k, Resistor_SMD:R_0805_2012Metric_Pad1.20x1.40mm_HandSolder, F.Cu at (256.4, 159.3)
- added R64: 3, Resistor_SMD:R_0805_2012Metric_Pad1.20x1.40mm_HandSolder, F.Cu at (256.4, 162.3)
- added R65: 3, Resistor_SMD:R_0805_2012Metric_Pad1.20x1.40mm_HandSolder, F.Cu at (256.4, 165.2)
- added R66: 10k, Resistor_SMD:R_0805_2012Metric_Pad1.20x1.40mm_HandSolder, F.Cu at (256.4, 168.2)
- added R67: 10k, Resistor_SMD:R_0805_2012Metric_Pad1.20x1.40mm_HandSolder, F.Cu at (256.4, 171.1)
- added R68: 560, Resistor_SMD:R_0805_2012Metric_Pad1.20x1.40mm_HandSolder, F.Cu at (256.4, 174.1)
- added R69: 1k, Resistor_SMD:R_0805_2012Metric_Pad1.20x1.40mm_HandSolder, F.Cu at (256.4, 177.0)
- moved D1 62.8 mm to (153.3, 147.2)
- moved C1 49.0 mm to (124.6, 143.6)
- moved C12 49.0 mm to (124.6, 146.6)
- moved C2 49.0 mm to (124.6, 137.6)
- moved C5 49.0 mm to (124.6, 134.6)
- moved R2 49.0 mm to (119.8, 124.7)
- moved R5 49.0 mm to (119.8, 127.7)
- moved R6 49.0 mm to (119.8, 133.6)
- moved R9 49.0 mm to (119.8, 142.4)
- moved Y1 49.0 mm to (132.9, 123.7)
- moved C3 49.0 mm to (124.6, 140.6)
- moved C8 49.0 mm to (124.6, 128.5)
- moved C9 49.0 mm to (124.6, 131.5)
- moved R1 49.0 mm to (119.8, 121.8)
- moved R3 49.0 mm to (119.8, 145.3)
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- renumbered C6 to C1, C7 to C12, C4 to C2, C5 to C3, C3 to C5, C1 to C8, C2 to C9, R9 to R3, R3 to R5, R5 to R6, R6 to R7, R7 to R8, R8 to R9, U1 to U2, U2 to U3
Connections:
- D1 pad 11: unconnected-(D1-Q0-Pad11) -> GND
- D1 pad 12: unconnected-(D1-Q11-Pad12) -> Net-(D1-1Y)
- D1 pad 13: unconnected-(D1-Q10-Pad13) -> GND
- D1 pad 3: G1H -> Net-(D1-2A)
- D1 pad 4: Net-(U2-Q2) -> Net-(D1-2B)
- D1 pad 5: Net-(D2-1B) -> GND
- D1 pad 6: G2H -> Net-(D1-2Y)
- D1 pad 8: G3H -> Net-(D1-3Y)
- U3 pad 4: Net-(U2-Q2) -> Net-(D1-2A)
- U3 pad 7: Net-(D2-1B) -> Net-(D1-2B)
Other:
- board outline removed

Commit message: VER1.0: начал раскидку компонентов на плате
Parts:
- removed the C15 at (238.0, 136.5)
- removed the C16 at (238.0, 139.8)
- removed the C20 at (158.1, 160.7)
- removed the C42 at (244.0, 136.5)
- removed the C43 at (244.0, 139.8)
- removed the C53 at (250.0, 136.5)
- removed the C54 at (250.0, 139.8)
- removed the C64 at (256.0, 136.5)
- removed the C65 at (256.0, 139.8)
- removed L11: 12u, Inductor_SMD:L_1210_3225Metric_Pad1.42x2.65mm_HandSolder
- removed L12: 47u, Inductor_SMD:L_1812_4532Metric_Pad1.30x3.40mm_HandSolder
- added C22: 4.7u, Capacitor_SMD:C_1206_3216Metric_Pad1.33x1.80mm_HandSolder, B.Cu at (338.8, 182.0)
- added C23: 100p, Capacitor_SMD:C_1206_3216Metric_Pad1.33x1.80mm_HandSolder, B.Cu at (341.2, 182.0)
- added C33: 4.7u, Capacitor_SMD:C_1206_3216Metric_Pad1.33x1.80mm_HandSolder, B.Cu at (335.8, 157.8)
- added C34: 4.7u, Capacitor_SMD:C_1206_3216Metric_Pad1.33x1.80mm_HandSolder, B.Cu at (338.8, 157.8)
- added C35: 100p, Capacitor_SMD:C_1206_3216Metric_Pad1.33x1.80mm_HandSolder, B.Cu at (341.2, 157.8)
- added C4: 100p, Capacitor_SMD:C_1206_3216Metric_Pad1.33x1.80mm_HandSolder, B.Cu at (341.2, 206.0)
- added C44: 680u, Capacitor_THT:CP_Radial_D13.0mm_P5.00mm, F.Cu at (335.2, 57.2)
- added C45: 4.7u, Capacitor_SMD:C_1206_3216Metric_Pad1.33x1.80mm_HandSolder, B.Cu at (338.5, 59.5)
- added C46: 10u, Capacitor_SMD:C_1206_3216Metric_Pad1.33x1.80mm_HandSolder, B.Cu at (347.5, 60.9)
- added C47: 22u, Capacitor_SMD:C_1206_3216Metric_Pad1.33x1.80mm_HandSolder, B.Cu at (352.8, 60.9)
- added C49: 4.7u, Capacitor_SMD:C_1206_3216Metric_Pad1.33x1.80mm_HandSolder, B.Cu at (335.8, 134.0)
- added C50: 4.7u, Capacitor_SMD:C_1206_3216Metric_Pad1.33x1.80mm_HandSolder, B.Cu at (338.8, 134.0)
- added C51: 100p, Capacitor_SMD:C_1206_3216Metric_Pad1.33x1.80mm_HandSolder, B.Cu at (341.2, 134.0)
- added C61: 4.7u, Capacitor_SMD:C_1206_3216Metric_Pad1.33x1.80mm_HandSolder, B.Cu at (335.8, 110.0)
- added C62: 4.7u, Capacitor_SMD:C_1206_3216Metric_Pad1.33x1.80mm_HandSolder, B.Cu at (338.8, 110.0)
- added C63: 100p, Capacitor_SMD:C_1206_3216Metric_Pad1.33x1.80mm_HandSolder, B.Cu at (341.2, 110.0)
- added C73: 4.7u, Capacitor_SMD:C_1206_3216Metric_Pad1.33x1.80mm_HandSolder, B.Cu at (335.8, 85.8)
- added C74: 4.7u, Capacitor_SMD:C_1206_3216Metric_Pad1.33x1.80mm_HandSolder, B.Cu at (338.8, 85.8)
- added C75: 100p, Capacitor_SMD:C_1206_3216Metric_Pad1.33x1.80mm_HandSolder, B.Cu at (341.2, 85.8)
- added C85: 4.7u, Capacitor_SMD:C_1206_3216Metric_Pad1.33x1.80mm_HandSolder, B.Cu at (319.5, 59.5)
- added C86: 10u, Capacitor_SMD:C_1206_3216Metric_Pad1.33x1.80mm_HandSolder, B.Cu at (313.1, 59.5)
- added C87: 330u, Capacitor_THT:CP_Radial_D10.0mm_P5.00mm, F.Cu at (322.8, 57.1)
- added C88: 10u, Capacitor_SMD:C_1206_3216Metric_Pad1.33x1.80mm_HandSolder, F.Cu at (294.4, 174.6)
- added C89: 100u, Capacitor_THT:CP_Radial_D5.0mm_P2.00mm, F.Cu at (299.8, 169.4)
- added C90: 56p, Capacitor_SMD:C_0805_2012Metric_Pad1.18x1.45mm_HandSolder, F.Cu at (342.0, 190.5)
- added D1: QA151C3, MORNSUN_my:QAxCx, F.Cu at (351.4, 206.0)
- added D11: QA151C3, MORNSUN_my:QAxCx, F.Cu at (351.4, 182.0)
- added D18: QA151C3, MORNSUN_my:QAxCx, F.Cu at (351.4, 158.0)
- added D24: K7815-1000R3, MORNSUN_my:K78xx-1000R3, F.Cu at (351.5, 60.4)
- added D26: QA151C3, MORNSUN_my:QAxCx, F.Cu at (351.4, 134.0)
- added D33: QA151C3, MORNSUN_my:QAxCx, F.Cu at (351.4, 110.0)
- added D40: QA151C3, MORNSUN_my:QAxCx, F.Cu at (351.4, 86.0)
- added D47: ~, LED_SMD:LED_0805_2012Metric_Pad1.15x1.40mm_HandSolder, F.Cu at (360.0, 57.8)
- added D48: WRB2405S-1WR2, MORNSUN_my:WRB_S-1WR2, F.Cu at (305.3, 62.3)
- added D49: ~, LED_SMD:LED_0805_2012Metric_Pad1.15x1.40mm_HandSolder, F.Cu at (291.5, 57.8)
- added F1: 0466002.NR, Fuse:Fuse_1206_3216Metric, F.Cu at (139.2, 164.2)
- added F2: 0466002.NR, Fuse:Fuse_1206_3216Metric, F.Cu at (294.2, 177.9)
- added R70: 3k, Resistor_SMD:R_0805_2012Metric_Pad1.20x1.40mm_HandSolder, F.Cu at (360.0, 63.0)
- added R71: 1k, Resistor_SMD:R_0805_2012Metric_Pad1.20x1.40mm_HandSolder, F.Cu at (291.5, 63.0)
- added R72: 120, Resistor_SMD:R_0805_2012Metric_Pad1.20x1.40mm_HandSolder, F.Cu at (342.0, 188.2)
- C17: renamed from C18; moved to B.Cu
- C18: renamed from C19; moved to B.Cu
- C2: renamed from C6; moved to B.Cu
- C21: moved to B.Cu
- C3: renamed from C7; moved to B.Cu
- C5: renamed from C10; moved to B.Cu
- C6: renamed from C11; moved to B.Cu
- L1, L3, L7, L9: value 12u -> 22u; moved to B.Cu
- L10: value 47u -> 4.7u; footprint Inductor_SMD:L_1812_4532Metric_Pad1.30x3.40mm_HandSolder -> Inductor_SMD:L_APV_ANR4030; moved to B.Cu
- L2, L8: value 47u -> 22u; footprint Inductor_SMD:L_1812_4532Metric_Pad1.30x3.40mm_HandSolder -> Inductor_SMD:L_1210_3225Metric_Pad1.42x2.65mm_HandSolder; moved to B.Cu
- L4: footprint Inductor_SMD:L_1812_4532Metric_Pad1.30x3.40mm_HandSolder -> Inductor_SMD:L_Vishay_IHLP-2525
- L5: value 12u -> 47u; footprint Inductor_SMD:L_1210_3225Metric_Pad1.42x2.65mm_HandSolder -> Inductor_SMD:L_Vishay_IHLP-2525
- L6: value 47u -> 12u; footprint Inductor_SMD:L_1812_4532Metric_Pad1.30x3.40mm_HandSolder -> Inductor_SMD:L_APV_ANR4030; moved to B.Cu
- R24: renamed from R23; footprint Resistor_SMD:R_0805_2012Metric_Pad1.20x1.40mm_HandSolder -> Resistor_SMD:R_2512_6332Metric_Pad1.40x3.35mm_HandSolder
- R25: renamed from R24; footprint Resistor_SMD:R_0805_2012Metric_Pad1.20x1.40mm_HandSolder -> Resistor_SMD:R_2512_6332Metric_Pad1.40x3.35mm_HandSolder
- R34, R35, R44, R45, R54, R55, R64, R65: footprint Resistor_SMD:R_0805_2012Metric_Pad1.20x1.40mm_HandSolder -> Resistor_SMD:R_2512_6332Metric_Pad1.40x3.35mm_HandSolder
- R6: renamed from R13; footprint Resistor_SMD:R_0805_2012Metric_Pad1.20x1.40mm_HandSolder -> Resistor_SMD:R_2512_6332Metric_Pad1.40x3.35mm_HandSolder
- R9: renamed from R14; footprint Resistor_SMD:R_0805_2012Metric_Pad1.20x1.40mm_HandSolder -> Resistor_SMD:R_2512_6332Metric_Pad1.40x3.35mm_HandSolder
- moved Q1 245.0 mm to (386.1, 188.6), turned to -90 degrees
- moved Q2 221.9 mm to (386.1, 164.6), turned to -90 degrees
- moved D4 220.0 mm to (389.2, 205.8), turned to 180 degrees
- moved D5 217.9 mm to (392.5, 197.0), turned to -90 degrees
- moved C6 212.4 mm to (362.0, 196.6), turned to -90 degrees
- moved C5 210.5 mm to (359.5, 196.6), turned to -90 degrees
- moved C18 206.7 mm to (362.0, 191.5), turned to -90 degrees
- moved C17 204.9 mm to (359.5, 191.5), turned to -90 degrees
- moved R4 199.9 mm to (381.5, 205.8), turned to 180 degrees
- moved C16 198.0 mm to (379.5, 198.2), turned to -90 degrees
- moved R13 195.1 mm to (381.8, 198.2), turned to 90 degrees
- moved R3 195.0 mm to (375.5, 205.8)
- moved C3 192.9 mm to (338.8, 206.0), turned to -90 degrees
- moved R6 191.1 mm to (376.5, 192.8)
- moved C2 190.9 mm to (335.8, 206.0), turned to -90 degrees
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- renumbered C4 to C10, C5 to C11, C14 to C12, C8 to C13, C9 to C14, C31 to C15, C17 to C16, C12 to C19, C32 to C20, C22 to C24, C23 to C25, C24 to C26, C25 to C27, C26 to C28, C28 to C29, C29 to C30, C30 to C31, C27 to C32, C33 to C36, C34 to C37, C35 to C38, C36 to C39, C37 to C40, C38 to C41, C39 to C42, C40 to C43, C41 to C48, C44 to C52, C45 to C53, C46 to C54, C47 to C55, C48 to C56, C49 to C57, C50 to C58, C51 to C59, C52 to C60, C55 to C64, C56 to C65, C57 to C66, C58 to C67, C59 to C68, C60 to C69, C2 to C7, C61 to C70, C62 to C71, C63 to C72, C66 to C76, C67 to C77, C68 to C78, C69 to C79, C3 to C8, C70 to C80, C71 to C81, C72 to C82, C73 to C83, C74 to C84, C13 to C9, D7 to D10, D16 to D15, D15 to D16, D10 to D19, D1 to D2, D24 to D25, D26 to D27, D27 to D28, D28 to D29, D4 to D3, D29 to D30, D30 to D31, D31 to D32, D33 to D34, D34 to D35, D35 to D36, D36 to D37, D37 to D38, D38 to D39, D5 to D4, D40 to D41, D41 to D42, D42 to D43, D43 to D44, D44 to D45, D45 to D46, D6 to D5, D18 to D6, D8 to D7, D3 to D8, D19 to D9, R31 to R10, R4 to R11, R5 to R12, R19 to R13, R6 to R14, R32 to R15, R7 to R16, R8 to R17, R33 to R18, R9 to R19, R10 to R2, R27 to R23, R29 to R27, R25 to R29, R11 to R3, R15 to R30, R16 to R31, R17 to R32, R18 to R33, R12 to R4, R30 to R5, R2 to R7, R3 to R8
Connections:
- net GND1 renamed GND_IN
- net Net-(D7-2C) renamed Q6
- C21 pad 1: Net-(C21-Pad1) -> +15V
- C24 pad 2: +15VL -> +15V_L1
- C25 pad 2: +15VL -> +15V_L1
- C3 pad 1: Net-(C7-Pad1) -> Net-(D1-Vin)
- C30 pad 1: -15VL -> -4V_L1
- C31 pad 1: -15VL -> -4V_L1
- C36 pad 1: A -> B
- C36 pad 2: +15V_H1 -> +15V_H2
- C37 pad 1: A -> B
- C37 pad 2: +15V_H1 -> +15V_H2
- C39 pad 1: A -> B
- C41 pad 2: A -> B
- C42 pad 1: -4V_H1 -> -4V_H2
- C42 pad 2: A -> B
- C43 pad 1: -4V_H1 -> -4V_H2
- C43 pad 2: A -> B
- C52 pad 2: +15VL -> +15V_L2
- C53 pad 2: +15VL -> +15V_L2
- C58 pad 1: -15VL -> -4V_L2
- C59 pad 1: -15VL -> -4V_L2
- C64 pad 1: A -> C
- C64 pad 2: +15V_H1 -> +15V_H3
- C65 pad 1: A -> C
- C65 pad 2: +15V_H1 -> +15V_H3
- C67 pad 1: A -> C
- C69 pad 2: A -> C
- C70 pad 1: -4V_H1 -> -4V_H3
- C70 pad 2: A -> C
- C71 pad 1: -4V_H1 -> -4V_H3
- C71 pad 2: A -> C
- C76 pad 2: +15VL -> +15V_L3
- C77 pad 2: +15VL -> +15V_L3
- C82 pad 1: -15VL -> -4V_L3
- C83 pad 1: -15VL -> -4V_L3
- D10 pad 1: Net-(D1-3A) -> Q3
- D10 pad 10: Net-(D1-1B) -> Q2
- D10 pad 2: Net-(D1-2B) -> Q4
- D10 pad 3: Net-(D1-3B) -> Q0
- D10 pad 4: Net-(D1-1A) -> Q5
- D10 pad 9: Net-(D1-2A) -> Q1
- D12 pad 1: -15VL -> -4V_L1
- D12 pad 10: PWM_N -> G1L
- D12 pad 11: PWM_P -> GND
- D12 pad 5: +15VL -> +15V_L1
- D12 pad 8: -15VL -> -4V_L1
- D19 pad 1: -4V_H1 -> -4V_H2
- D19 pad 10: PWM_N -> G2H
- D19 pad 11: PWM_P -> GND
- D19 pad 3: A -> B
- D19 pad 5: +15V_H1 -> +15V_H2
- D19 pad 8: -4V_H1 -> -4V_H2
- D2 pad 1: Net-(D1-1A) -> Q0
- D2 pad 10: Net-(D1-3B) -> Q5
- D2 pad 2: Net-(D1-1B) -> Q1
- D2 pad 3: Net-(D1-2A) -> Q2
- D2 pad 4: Net-(D1-2B) -> Q3
- D2 pad 9: Net-(D1-3A) -> Q4
- D23 pad 2: A -> B
- D27 pad 1: -15VL -> -4V_L2
- D27 pad 10: PWM_N -> G2L
- D27 pad 11: PWM_P -> GND
- D27 pad 5: +15VL -> +15V_L2
- D27 pad 8: -15VL -> -4V_L2
- D29 pad 1: A -> B
- D3 pad 10: PWM_N -> G1H
- D3 pad 11: PWM_P -> GND
- D34 pad 1: -4V_H1 -> -4V_H3
- D34 pad 10: PWM_N -> G3H
- D34 pad 11: PWM_P -> GND
- D34 pad 3: A -> C
- D34 pad 5: +15V_H1 -> +15V_H3
- D34 pad 8: -4V_H1 -> -4V_H3
- D38 pad 2: A -> C
- D41 pad 1: -15VL -> -4V_L3
- D41 pad 10: PWM_N -> G3L
- D41 pad 11: PWM_P -> GND
- D41 pad 5: +15VL -> +15V_L3
- D41 pad 8: -15VL -> -4V_L3
- D43 pad 1: A -> C
- D8 pad 2: G1H -> Net-(D8-1Y)
- L1 pad 2: Net-(C7-Pad1) -> Net-(D1-Vin)
- L10 pad 1: Net-(C54-Pad1) -> Net-(D48-Vin)
- L2 pad 1: Net-(C7-Pad1) -> +15V
- L3 pad 2: Net-(C21-Pad1) -> Net-(D18-Vin)
- L4 pad 1: Net-(C21-Pad1) -> Net-(F1-Pad2)
- L4 pad 2: Net-(D11-Vin) (its old number) -> Net-(L4-Pad2)
- L5 pad 1: +15V -> Net-(L4-Pad2)
- L7 pad 2: Net-(C43-Pad1) -> Net-(D26-Vin)
- L8 pad 1: Net-(C43-Pad1) -> +15V
- L9 pad 2: Net-(C54-Pad1) -> Net-(D40-Vin)
- Q3 pad 3: A -> B
- Q4 pad 2: A -> B
- Q5 pad 3: A -> C
- Q6 pad 2: A -> C
- R20 pad 2: +15VL -> +15V_L1
- R30 pad 2: +15V_H1 -> +15V_H2
- R37 pad 1: A -> B
- R40 pad 2: +15VL -> +15V_L2
- R50 pad 2: +15V_H1 -> +15V_H3
- R57 pad 1: A -> C
- R60 pad 2: +15VL -> +15V_L3
- U3 pad 1: Net-(D1-3B) -> Q5
- U3 pad 10: Net-(D1-3A) -> Q4
- U3 pad 2: Net-(D1-1B) -> Q1
- U3 pad 3: Net-(D1-1A) -> Q0
- U3 pad 4: Net-(D1-2A) -> Q2
- U3 pad 7: Net-(D1-2B) -> Q3
Routing:
- net Net-(D3-~{FLT}): track 0.00 -> 26.0 mm
- net Net-(D3-OUTH): track 0.00 -> 20.0 mm
- net Net-(D3-OUTL): track 0.00 -> 18.8 mm
- net Net-(D3-RDY): track 0.00 -> 12.8 mm
- net GateH1: track 0.00 -> 10.8 mm
- net G1H: track 0.00 -> 3.89 mm
- net Net-(D9-A): track 0.00 -> 2.26 mm
- net Net-(D6-A): track 0.00 -> 2.26 mm
Other:
- copper layers 2 -> 4
